Commit message: Add leap_motion_link tf

File: urdf/kinect_with_leap.urdf.xacro (robot description, xacro)
@@ -1,7 +1,8 @@
 <?xml version="1.0"?>
-<robot name="teaching_base" xmlns:xacro="http://ros.org/wiki/xacro">
+<robot name="teaching_booth" xmlns:xacro="http://ros.org/wiki/xacro">
   <xacro:include filename="$(find kinect_bringup)/urdf/common.xacro" />
   <xacro:include filename="$(find kinect_bringup)/urdf/sensor/kinect.urdf.xacro"/>
   <xacro:include filename="$(find kinect_bringup)/urdf/sensor/kinect.gazebo.xacro"/>
+  <!-- <xacro:include filename="$(find kinect_with_leap)/urdf/leap.urdf.xacro"/> -->
   <link name="world"/>
   <!-- add Kinect V2 -->
@@ -42,3 +43,12 @@
   <!-- Gazebo -->
   <!-- <xacro:kinect_gazebo name="kinect_side"/> -->
+  <!-- Add Leap Motion -->
+  <!-- Link -->
+  <link name="leap_motion_link"/>
+  <!-- Joint -->
+  <joint name="leap_motion_joint" type="fixed">
+    <origin xyz="0.057 0 0.565" rpy="${M_PI/2} ${M_PI} 0"/>
+    <parent link="world"/>
+    <child link="leap_motion_link"/>
+  </joint>
 </robot>

Commit message: Modified kinect position

File: urdf/kinect_with_leap.urdf.xacro (robot description, xacro)
@@ -14,5 +14,5 @@
   <joint name="joint_kinect" type="fixed">
     <!-- <origin xyz="0.15 0.38 0.9368" rpy="3.1416 1.5024 3.1416" /> -->
-    <origin xyz="1.28 0 0.5" rpy="0 0.3982 -3.123" />
+    <origin xyz="-0.0243 -0.0348 1.0267" rpy="0.3036 1.5239 0.3282" />
     <parent link="world"/>
     <child link="kinect"/>
@@ -48,5 +48,5 @@
   <!-- Joint -->
   <joint name="leap_motion_joint" type="fixed">
-    <origin xyz="0.057 0 0.565" rpy="${M_PI/2} ${M_PI} 0"/>
+    <origin xyz="-0.0243 -0.0348 0.5" rpy="${M_PI/2} ${M_PI} 0"/>
     <parent link="world"/>
     <child link="leap_motion_link"/>
